Commit message: Aragog

File: Hardware/Aragog/urdf/Aragog.urdf (robot description, URDF)
Before this commit: robot Aragog URDF part 2, 4 links, 3 joints
Links:
- link base_link: geometry collision mesh filename=package://Aragog/meshes/base_link.STL; visual mesh filename=package://Aragog/meshes/base_link.STL
- link left_leg: mass 0.0099613 -> 0.099613; geometry collision mesh filename=package://Aragog/meshes/left_leg.STL; visual mesh filename=package://Aragog/meshes/left_leg.STL
- link middle_leg: mass 0.0064836 -> 0.064836; geometry collision mesh filename=package://Aragog/meshes/middle_leg.STL; visual mesh filename=package://Aragog/meshes/middle_leg.STL
- link right_leg: mass 0.0099613 -> 0.099613; geometry collision mesh filename=package://Aragog/meshes/right_leg.STL; visual mesh filename=package://Aragog/meshes/right_leg.STL
Joints:
- joint left_revolute: limit lower=0 upper=2 effort=0 velocity=0 -> lower=0 upper=3.14 effort=0.1 velocity=0
- joint middle_revolute: limit lower=0 upper=2 effort=0 velocity=0 -> lower=0 upper=3.14 effort=0.1 velocity=0
- joint right_revolute: limit lower=0 upper=2 effort=0 velocity=0 -> lower=0 upper=3.14 effort=0.1 velocity=0

Commit message: karthiks1701

File: Hardware/Aragog/urdf/Aragog.urdf (robot description, URDF)
Before this commit: robot Aragog, 4 links, 3 joints
Joints:
- joint left_revolute: limit lower=0 upper=3.14 effort=0.1 velocity=0 -> lower=-3.14 upper=3.14 effort=0.5 velocity=0
- joint middle_revolute: limit lower=0 upper=3.14 effort=0.1 velocity=0 -> lower=-3.14 upper=3.14 effort=0.5 velocity=0
- joint right_revolute: limit lower=0 upper=3.14 effort=0.1 velocity=0 -> lower=-3.14 upper=3.14 effort=0.5 velocity=0
